File: eagle/B4L_power_PCB.sch (EAGLE design)
At the start: 39 parts, among them IC1 LM2576S, IC2 TL081CP, Q1 STP40NF03L, U1 TMC2209-LA

Commit message: Update PCB power for 48V supply
Parts:
- removed C11, C5, C6: 100nF, rcl:C-EUC0603
- removed C12, C8: 4.7uF, rcl:C-EUC0603
- removed C4: 22nF, rcl:C-EUC0603
- removed C7: 10uF, rcl:C-EUC0603
- removed IC2: TL081CP, custom:TL081D
- removed R10, R11: 0.11, rcl:R-US_R0603
- removed R3: 56k, rcl:R-US_R0603
- removed R4: 100k, rcl:R-US_R0603
- removed U$1: EEEFK1H102AM, custom:EEEFK1H102AM
- removed U1: TMC2209-LA, custom:TMC2209-LA
- added IC3: LM211PSOIC, custom:LM211PSOIC
- added JP6: (no value), pinhead:PINHD-1X2
- added LED1: (no value), led:LED3MM
- C1: device Panasonic-EEEFT_EEEH:EEE-FTH101XAP-CASE-D8 -> custom:EEV-EB2D101M-CASE-K21
- C3: value 100nF -> 470uF; device rcl:C-EUC0603 -> custom:EEVFK1K471M-CASE-K16
- C9: device rcl:C-EUC0603 -> rcl:C-EUC1206
- D1, D3: value MBRA340T3G -> B360A-13-F; device custom:MBRA340T3G -> custom:B360A-13-F
- D2: value MBRA340T3G -> ES1A+; device custom:MBRA340T3G -> custom:ESIA+
- F1: value MST 4A 250V -> MCCFB2410TTT/4
- IC1: value LM2576S -> LM2576HVS-12; device custom:LM2576S -> custom:LM2576HVS
- JP2: device pinhead:PINHD-1X8 -> pinhead:PINHD-1X2
- JP3: device pinhead:PINHD-1X14 -> pinhead:PINHD-1X2
- Q1: value STP40NF03L -> SI2356DS-T1-GE3
- R2: value 100k -> 1k
- R6, R8, R9: value 20k -> 100k
- R7: value 20k -> 56k
Connections:
- net SUPPLY-24VDC renamed SUPPLY-48VDC
- removed net 24VDC: C1.1, C3.2, C5.1, C6.1, C7.1, C9.1, F1.2, IC1.VIN, R1.2, U$1.1, U1B.VS, U1B.VS_2
- removed net ARD-5VDC: C12.1, JP3.4, U1B.VCC_IO
- removed net MOTOR-DIAG: JP3.12, U1A.DIAG
- removed net MOTOR-DIR: JP3.5, U1A.DIR
- removed net MOTOR-EN: JP3.7, R8.1, U1A.ENN
- removed net MOTOR-INDEX: JP3.11, U1A.INDEX
- removed net MOTOR-SPRD: JP3.13, U1A.SPREAD
- removed net MOTOR-STEP: JP3.6, U1A.STEP
- removed net MOTOR-UART: JP3.10, JP3.9, R9.2, U1A.PDN_UART
- removed net MOTOR_A: JP2.1, U1A.OA1
- removed net MOTOR_B: JP2.5, U1A.OB1
- removed net MOTOR_C: JP2.4, U1A.OA2
- removed net MOTOR_D: JP2.8, U1A.OB2
- removed net N$10: R11.1, U1A.BRB
- removed net N$12: JP2.6, JP2.7
- removed net N$5: IC2.OUT, R2.2
- removed net N$6: R6.2, R7.2, U1B.VREF
- removed net N$7: C4.2, U1A.CPO
- removed net N$8: JP2.2, JP2.3
- removed net N$9: R10.1, U1A.BRA
- removed net TMC-5VDC: C8.1, R6.1, R8.2, U1A.5VOUT
- removed net TMC-CPI: C4.1, U1A.CPI
- new net 48VDC: C1.1, C3.1, C9.1, F1.2, IC1.VIN, JP6.1, R1.2
- net 12VDC: now also IC3.VCC+, R2.1, R7.1, R9.1; no longer R3.1
- net AUX_PWR_CHK: now also IC3.COLOUT, JP3.2, R9.2; no longer JP3.3, R2.1
- net BATT-9VDC: now also IC3.IN+, R6.1; no longer IC2.+IN
- net GND: now also C3.2, IC3.EMITOUT, IC3.VCC-, JP2.2, JP6.2, LED1.C, R6.2, R8.2; no longer C11.2, C12.2, C5.2, C6.2, C7.2, C8.2, IC2.V-, JP3.14, R10.2, R11.2, R4.2, R7.1, R9.1, U$1.2, U1A.CLK, U1A.EPAD, U1A.MS1_AD0, U1A.MS2_AD1, U1A.STDBY, U1B.GND, U1B.GND_2
- net MAIN_PWR_CHK: now also JP3.1; no longer JP3.2
- net N$3: now also LED1.A, R2.2; no longer IC2.-IN, R3.2, R4.1
- net N$4: now also IC3.IN-, R7.2, R8.1; no longer C3.1, U1B.VCP
- net VOUT-12/9VDC: now also JP2.1; no longer C11.1, IC2.V+, JP3.1
Other:
- note added: "DC/DC 48->12V"
- note added: "Power-on LED"
- note added: "to UI board"
- note added: "to motor driver"
- note removed: "DC/DC 24->12V"
- note removed: "to Arduino"
- note removed: "to motor"
